File: rs232_usb.brd (EAGLE design)
At the start: 40 x 40 mm, 17 parts, among them IC1 FT232RL, T1 BC847

Commit message: 1. Fertiges Layout (Beidseitig)
Parts:
- moved X1 24.6 mm to (8.38, 4.83)
- moved 3V3 22.6 mm to (6.10, 33.0), flipped to the bottom
- moved 5V 22.6 mm to (2.79, 33.0), flipped to the bottom
- moved U1 22.2 mm to (8.38, 18.0), turned to 90 degrees
- moved TS1 22.2 mm to (8.38, 26.9), flipped to the bottom, turned to 0 degrees
- moved R2 21.0 mm to (3.30, 20.8), flipped to the bottom
- moved C3 17.4 mm to (8.38, 12.2), flipped to the bottom
- moved LED2 15.9 mm to (11.4, 19.1), flipped to the bottom
- moved LED1 15.9 mm to (11.4, 15.7), flipped to the bottom
- moved BT1 15.8 mm to (8.38, 36.3), turned to 180 degrees
- moved R1 15.5 mm to (9.65, 34.0), flipped to the bottom, turned to 0 degrees
- moved C1 14.5 mm to (9.65, 31.8), flipped to the bottom
- moved R3 13.2 mm to (7.62, 15.7), flipped to the bottom
- moved R4 13.2 mm to (7.37, 19.1), flipped to the bottom
- moved C2 12.8 mm to (10.9, 22.4), flipped to the bottom
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Routing:
- net +3V3: track 102.6 -> 26.6 mm, vias 0 -> 1
- net +5V: track 23.8 -> 70.3 mm, vias 0 -> 5
- net LED2: track 40.0 -> 12.0 mm, vias 0 -> 1
- net LED1: track 42.2 -> 18.8 mm, vias 0 -> 1
- net RXD_5V: track 34.4 -> 17.1 mm
- net TXD_BT_3V3: track 34.7 -> 18.9 mm, vias 0 -> 1
- net TXD_5V: track 35.0 -> 21.5 mm
- net RESET: track 21.6 -> 8.50 mm, vias 0 -> 1
- net RXD_BT: track 36.9 -> 25.5 mm, vias 0 -> 2
- net N$1: track 11.5 -> 5.75 mm
- net TXD_BT: track 4.02 -> 8.49 mm
- net USB_5V_P: track 8.16 -> 11.2 mm
- net USB_5V_N: track 8.25 -> 11.2 mm
- net N$7: track 6.42 -> 4.85 mm
- net USB_3V3_N: track 15.1 -> 16.0 mm
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- added copper zone on layer 16, net GND
Other:
- board size 40 x 40 mm -> 17 x 40 mm

Commit message: added Readme
Routing:
- net +5V: track 70.3 -> 81.5 mm
Changed lines of the file:
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@@
 <setting verticaltext="up"/>
 </settings>
-<grid distance="0.01" unitdist="inch" unit="mm" style="lines" multiple="1" display="yes" altdistance="0.005" altunitdist="inch" altunit="inch"/>
+<grid distance="0.01" unitdist="inch" unit="inch" style="lines" multiple="1" display="yes" altdistance="0.005" altunitdist="inch" altunit="inch"/>
 <layers>
 <layer number="1" name="Top" color="4" fill="1" visible="yes" active="yes"/>
@@
 <wire x1="6.782" y1="10.16" x2="3.81" y2="10.16" width="0.4064" layer="1"/>
 <wire x1="3.81" y1="10.16" x2="1.27" y2="12.7" width="0.4064" layer="1"/>
-<wire x1="3.302" y1="19.978" x2="1.27" y2="19.978" width="0.254" layer="16"/>
-<wire x1="1.27" y1="19.978" x2="1.27" y2="15.748" width="0.254" layer="16"/>
+<wire x1="3.302" y1="19.978" x2="1.27" y2="19.978" width="0.4064" layer="16"/>
 <via x="1.27" y="15.748" extent="1-16" drill="0.6096" shape="octagon"/>
+<wire x1="1.27" y1="19.978" x2="1.27" y2="15.748" width="0.4064" layer="16"/>
 <wire x1="5.4642" y1="15.748" x2="5.4642" y2="15.759" width="0.254" layer="1"/>
-<wire x1="1.27" y1="15.748" x2="1.27" y2="12.7" width="0.254" layer="1"/>
+<wire x1="1.27" y1="15.748" x2="1.27" y2="12.7" width="0.4064" layer="1"/>
 <wire x1="5.857" y1="12.192" x2="4.064" y2="12.192" width="0.254" layer="16"/>
 <wire x1="4.064" y1="12.192" x2="1.27" y2="14.986" width="0.254" layer="16"/>
@@
 <wire x1="5.857" y1="12.192" x2="5.857" y2="13.731" width="0.254" layer="16"/>
 <wire x1="5.857" y1="13.731" x2="6.35" y2="14.224" width="0.254" layer="16"/>
-<wire x1="4.757" y1="29.707" x2="2.551" y2="29.707" width="0.254" layer="1"/>
-<wire x1="2.551" y1="29.707" x2="2.286" y2="29.972" width="0.254" layer="1"/>
+<wire x1="4.757" y1="29.707" x2="2.551" y2="29.707" width="0.4064" layer="1"/>
+<wire x1="2.551" y1="29.707" x2="2.286" y2="29.972" width="0.4064" layer="1"/>
 <via x="2.286" y="29.972" extent="1-16" drill="0.6096" shape="octagon"/>
-<wire x1="2.286" y1="29.972" x2="2.286" y2="31.662" width="0.254" layer="16"/>
 <wire x1="2.286" y1="31.662" x2="2.794" y2="32.17" width="0.254" layer="16"/>
-<wire x1="4.757" y1="29.707" x2="9.133" y2="29.707" width="0.254" layer="1"/>
+<wire x1="4.757" y1="29.707" x2="9.133" y2="29.707" width="0.4064" layer="1"/>
 <wire x1="9.133" y1="29.707" x2="9.144" y2="29.718" width="0.254" layer="1"/>
 <via x="14.224" y="27.686" extent="1-16" drill="0.6096" shape="octagon"/>
@@
 <wire x1="13.503" y1="26.457" x2="12.007" y2="26.457" width="0.254" layer="1"/>
 <wire x1="14.224" y1="27.686" x2="13.97" y2="27.94" width="0.254" layer="16"/>
-<wire x1="13.97" y1="27.94" x2="10.9" y2="27.94" width="0.254" layer="16"/>
-<wire x1="10.9" y1="27.94" x2="9.133" y2="29.707" width="0.254" layer="16"/>
+<wire x1="13.97" y1="27.94" x2="10.9" y2="27.94" width="0.4064" layer="16"/>
+<wire x1="10.9" y1="27.94" x2="9.133" y2="29.707" width="0.4064" layer="16"/>
 <via x="9.133" y="29.707" extent="1-16" drill="0.6096" shape="octagon"/>
 <wire x1="11.772" y1="22.352" x2="13.462" y2="22.352" width="0.254" layer="16"/>
@@
 <wire x1="15.24" y1="25.4" x2="15.24" y2="26.67" width="0.254" layer="16"/>
 <wire x1="15.24" y1="26.67" x2="14.224" y2="27.686" width="0.254" layer="16"/>
+<wire x1="2.286" y1="29.972" x2="1.27" y2="28.956" width="0.4064" layer="16"/>
+<wire x1="1.27" y1="28.956" x2="1.27" y2="19.978" width="0.4064" layer="16"/>
+<wire x1="2.286" y1="29.972" x2="2.794" y2="30.48" width="0.4064" layer="16"/>
+<wire x1="2.794" y1="30.48" x2="2.794" y2="32.17" width="0.4064" layer="16"/>
 </signal>
 <signal name="USB_5V_P">
